Commit message: adding inertial properties for all links

File: URDF/urcbt.urdf (robot description, URDF)
Before this commit: robot URCBOT, 7 links, 6 joints
Links:
- link back_left_leg: mass None -> 1
- link back_right_leg: mass None -> 1
- link base_link: mass None -> 5
- link front_left_leg: mass None -> 1
- link front_right_leg: mass None -> 1
- link middle_left_leg: mass None -> 1
- link middle_right_leg: mass None -> 1

Commit message: adding limits to joints

File: URDF/urcbt.urdf (robot description, URDF)
Before this commit: robot URCBOT, 7 links, 6 joints
Links:
- link base_link: geometry visual box size=6.5 3.3 0.4
Joints:
- joint base_to_back_left_leg: limit (none) -> lower=-2.2 upper=0.7 effort=30 velocity=1.0
- joint base_to_back_right_leg: limit (none) -> lower=-2.2 upper=0.7 effort=30 velocity=1.0
- joint base_to_front_left_leg: limit (none) -> lower=-2.2 upper=0.7 effort=30 velocity=1.0
- joint base_to_front_right_leg: limit (none) -> lower=-2.2 upper=0.7 effort=30 velocity=1.0
- joint base_to_middle_left_leg: limit (none) -> lower=-2.2 upper=0.7 effort=30 velocity=1.0
- joint base_to_middle_right_leg: limit (none) -> lower=-2.2 upper=0.7 effort=30 velocity=1.0

Commit message: junk

File: URDF/urcbt.urdf (robot description, URDF)
Before this commit: robot URCBOT, 7 links, 6 joints
Joints:
- joint base_to_middle_left_leg: limit lower=-2.2 upper=0.7 effort=30 velocity=1.0 -> (none)

Commit message: camera_link and plugin

File: URDF/urcbt.urdf (robot description, URDF)
Before this commit: robot URCBOT, 7 links, 6 joints
Links:
- added link camera_link, mass 1e-5; collision box size=0.15 0.4 0.3; visual box size=0.15 0.4 0.3
Joints:
- added joint camera_joint: type fixed, parent base_link, child camera_link, origin xyz=3.0 0.0 0.32, axis 0 1 0

Commit message: adding collision properties to links

File: URDF/urcbt.urdf (robot description, URDF)
Before this commit: robot URCBOT, 8 links, 7 joints
Links:
- link back_left_leg: geometry collision cylinder length=0.50 radius=0.6; visual cylinder length=0.50 radius=0.6
- link back_right_leg: geometry collision cylinder length=0.50 radius=0.6; visual cylinder length=0.50 radius=0.6
- link base_link: geometry collision box size=6.5 3.3 0.4; visual box size=6.5 3.3 0.4
- link front_left_leg: geometry collision cylinder length=0.50 radius=0.6; visual cylinder length=0.50 radius=0.6
- link front_right_leg: geometry collision cylinder length=0.50 radius=0.6; visual cylinder length=0.50 radius=0.6
- link middle_left_leg: geometry collision cylinder length=0.50 radius=0.6; visual cylinder length=0.50 radius=0.6
- link middle_right_leg: geometry collision cylinder length=0.50 radius=0.6; visual cylinder length=0.50 radius=0.6
