Commit message: new package for simulation, with kinect plugin added

File: src/simulation/URDF/urcbt.urdf (robot description, URDF)
Before this commit: robot URCBOT, 8 links, 7 joints
Links:
- removed link camera_link
- added link kinect_link, mass 1e-5; collision box size=0.33 1.4 0.3; visual box size=0.33 1.4 0.3
Joints:
- removed joint camera_joint
- added joint kinect_joint: type fixed, parent base_link, child kinect_link, origin xyz=3.2 0.0 0.32, axis 0 1 0

Commit message: diff plugin

File: src/simulation/URDF/urcbt.urdf (robot description, URDF)
Before this commit: robot URCBOT, 8 links, 7 joints
Links:
- added link kinect_depth_frame, mass 0.0001
- added link kinect_depth_optical_frame, mass 0.0001
- link kinect_link: mass 1e-5 -> 0.0001; geometry visual box size=1.0 .5 0.2
Joints:
- added joint depth_optical_joint: type fixed, parent kinect_depth_frame, child kinect_depth_optical_frame, origin xyz=0 0 0 rpy=1.57075 0 1.57075
- added joint kinect_depth_joint: type fixed, parent kinect_link, child kinect_depth_frame, origin xyz=0 0.028 0 rpy=0 0 0
