Commit message: adding depth_image_to_laserscan

File: src/mybot_ws/src/mybot_description/urdf/mybot.xacro (robot description, xacro)
@@ -9,5 +9,5 @@
     <inertial>
       <mass value="15.0"/>
-      <origin xyz="0.0 0 0.1" rpy=" 0 0 0"/>
+      <origin xyz="0.0 0 0.0" rpy=" 0 0 0"/>
       <inertia
           ixx="0.1" ixy="0" ixz="0"
@@ -25,4 +25,5 @@
         <box size=".9 .6 .1"/>
       </geometry>
+      <material name="orange"/>
     </visual>
   </link>
@@ -39,5 +40,5 @@
         <box size="0.1 0.3 0.1"/>
       </geometry>
-      <material name="Red"/>
+      <material name="blue"/>
     </visual>
     <inertial>
@@ -60,4 +61,5 @@
         <cylinder radius="0.1" length="0.05"/>
       </geometry>
+      <material name="blue"/>
     </visual>
     <inertial>
@@ -83,4 +85,5 @@
         <cylinder radius="0.1" length="0.05"/>
       </geometry>
+      <material name="blue"/>
     </visual>
     <inertial>
@@ -106,4 +109,5 @@
         <cylinder radius="0.1" length="0.05"/>
       </geometry>
+      <material name="blue"/>
     </visual>
     <inertial>
@@ -129,4 +133,5 @@
         <cylinder radius="0.1" length="0.05"/>
       </geometry>
+      <material name="blue"/>
     </visual>
     <inertial>
@@ -152,4 +157,5 @@
         <cylinder radius="0.1" length="0.05"/>
       </geometry>
+      <material name="blue"/>
     </visual>
     <inertial>
@@ -175,4 +181,5 @@
         <cylinder radius="0.1" length="0.05"/>
       </geometry>
+      <material name="blue"/>
     </visual>
     <inertial>

Commit message: adding urdf

File: src/mybot_ws/src/mybot_description/urdf/mybot.xacro (robot description, xacro)
@@ -1,6 +1,6 @@
 <?xml version='1.0'?>
 <robot name="myrobot" xmlns:xacro="http://www.ros.org/wiki/xacro">
-  <xacro:property name="cameraSize" value="0.05"/>
-  <xacro:property name="cameraMass" value="0.1"/>
+  <!--xacro:property name="cameraSize" value="0.05"/>
+  <xacro:property name="cameraMass" value="0.1"/-->
   <xacro:include filename="$(find mybot_description)/urdf/mybot.gazebo" />
   <xacro:include filename="$(find mybot_description)/urdf/materials.xacro" />
@@ -9,21 +9,21 @@
     <pose>0 0 0 0 0 0</pose>
     <inertial>
-      <mass value="15.0"/>
-      <origin xyz="0.0 0 0.1" rpy=" 0 0 0"/>
-      <inertia
-          ixx="0.1" ixy="0" ixz="0"
-          iyy="0.1" iyz="0"
-          izz="0.1"
+      <mass value="47.0"/>
+      <origin xyz="0.0 0.0 0.0" rpy=" 0 0 0"/>
+      <inertia
+          ixx="1" ixy="0" ixz="0"
+          iyy="1" iyz="0"
+          izz="1"
       />
     </inertial>
     <collision name='collision'>
       <geometry>
-        <box size=".8 .4 .1"/>
+        <box size="1.4 0.96 0.505"/>
       </geometry>
     </collision>
     <visual name='chassis_visual'>
-      <origin xyz="0 0 0" rpy=" 0 0 0"/>
-      <geometry>
-        <box size=".8 .4 .1"/>
+      <origin xyz="0 0 0.505" rpy=" 0 0 0"/>
+      <geometry>
+        <box size="1.4 .96 .505"/>
       </geometry>
     </visual>
@@ -32,22 +32,22 @@
     <!--origin xyz="0.1 0.13 0.1" rpy="0 1.5707 1.5707"/-->
     <collision name="collision">
-      <origin xyz="0 0 0" rpy="0 1.5707 1.5707"/>
-      <geometry>
-        <cylinder radius="0.1" length="0.05"/>
+      <origin xyz="0.0 0.0 0.0" rpy="0 1.5707 1.5707"/>
+      <geometry>
+        <cylinder radius="0.125" length="0.150"/>
       </geometry>
     </collision>
     <visual name="left_wheel_visual">
-      <origin xyz="0 0 0" rpy="0 1.5707 1.5707"/>
-      <geometry>
-        <cylinder radius="0.1" length="0.05"/>
-      </geometry>
-    </visual>
-    <inertial>
-      <origin xyz="0 0 0" rpy="0 1.5707 1.5707"/>
-      <mass value="5"/>
-      <inertia
-        ixx=".1" ixy="0.0" ixz="0.0"
-        iyy=".1" iyz="0.0"
-        izz=".1"/>
+      <origin xyz="0.0 0.0 0.0" rpy="0 1.5707 1.5707"/>
+      <geometry>
+        <cylinder radius="0.125" length="0.150"/>
+      </geometry>
+    </visual>
+    <inertial>
+      <origin xyz="0.0 0.0 0.0" rpy="0 1.5707 1.5707"/>
+      <mass value="4"/>
+      <inertia
+        ixx="1" ixy="0.0" ixz="0.0"
+        iyy="1" iyz="0.0"
+        izz="1"/>
     </inertial>
   </link>
@@ -55,7 +55,7 @@
     <!--origin xyz="0.1 0.13 0.1" rpy="0 1.5707 1.5707"/-->
     <collision name="collision">
-      <origin xyz="0 0 0" rpy="0 1.5707 1.5707"/>
-      <geometry>
-        <cylinder radius="0.1" length="0.05"/>
+      <origin xyz=" 0 0 0" rpy="0 1.5707 1.5707"/>
+      <geometry>
+        <cylinder radius="0.125" length="0.150"/>
       </geometry>
     </collision>
@@ -63,14 +63,14 @@
       <origin xyz="0 0 0" rpy="0 1.5707 1.5707"/>
       <geometry>
-        <cylinder radius="0.1" length="0.05"/>
-      </geometry>
-    </visual>
-    <inertial>
-      <origin xyz="0 0 0" rpy="0 1.5707 1.5707"/>
-      <mass value="5"/>
-      <inertia
-        ixx=".1" ixy="0.0" ixz="0.0"
-        iyy=".1" iyz="0.0"
-        izz=".1"/>
+        <cylinder radius="0.125" length="0.150"/>
+      </geometry>
+    </visual>
+    <inertial>
+      <origin xyz="0 0 0" rpy="0 1.5707 1.5707"/>
+      <mass value="4"/>
+      <inertia
+        ixx="1" ixy="0.0" ixz="0.0"
+        iyy="1" iyz="0.0"
+        izz="1"/>
     </inertial>
   </link>
@@ -80,5 +80,5 @@
       <origin xyz="0 0 0" rpy="0 1.5707 1.5707"/>
       <geometry>
-        <cylinder radius="0.1" length="0.05"/>
+        <cylinder radius="0.125" length="0.150"/>
       </geometry>
     </collision>
@@ -86,14 +86,14 @@
       <origin xyz="0 0 0" rpy="0 1.5707 1.5707"/>
       <geometry>
-        <cylinder radius="0.1" length="0.05"/>
-      </geometry>
-    </visual>
-    <inertial>
-      <origin xyz="0 0 0" rpy="0 1.5707 1.5707"/>
-      <mass value="5"/>
-      <inertia
-        ixx=".1" ixy="0.0" ixz="0.0"
-        iyy=".1" iyz="0.0"
-        izz=".1"/>
+        <cylinder radius="0.125" length="0.150"/>
+      </geometry>
+    </visual>
+    <inertial>
+      <origin xyz="0 0 0" rpy="0 1.5707 1.5707"/>
+      <mass value="4"/>
+      <inertia
+        ixx="1" ixy="0.0" ixz="0.0"
+        iyy="1" iyz="0.0"
+        izz="1"/>
     </inertial>
   </link>
@@ -103,5 +103,5 @@
       <origin xyz="0 0 0" rpy="0 1.5707 1.5707"/>
       <geometry>
-        <cylinder radius="0.1" length="0.05"/>
+        <cylinder radius="0.125" length="0.150"/>
       </geometry>
     </collision>
@@ -109,14 +109,14 @@
       <origin xyz="0 0 0" rpy="0 1.5707 1.5707"/>
       <geometry>
-        <cylinder radius="0.1" length="0.05"/>
-      </geometry>
-    </visual>
-    <inertial>
-      <origin xyz="0 0 0" rpy="0 1.5707 1.5707"/>
-      <mass value="5"/>
-      <inertia
-        ixx=".1" ixy="0.0" ixz="0.0"
-        iyy=".1" iyz="0.0"
-        izz=".1"/>
+        <cylinder radius="0.125" length="0.150"/>
+      </geometry>
+    </visual>
+    <inertial>
+      <origin xyz="0 0 0" rpy="0 1.5707 1.5707"/>
+      <mass value="4"/>
+      <inertia
+        ixx="1" ixy="0.0" ixz="0.0"
+        iyy="1" iyz="0.0"
+        izz="1"/>
     </inertial>
   </link>
@@ -126,5 +126,5 @@
       <origin xyz="0 0 0" rpy="0 1.5707 1.5707"/>
       <geometry>
-        <cylinder radius="0.1" length="0.05"/>
+        <cylinder radius="0.125" length="0.150"/>
       </geometry>
     </collision>
@@ -132,14 +132,14 @@
       <origin xyz="0 0 0" rpy="0 1.5707 1.5707"/>
       <geometry>
-        <cylinder radius="0.1" length="0.05"/>
-      </geometry>
-    </visual>
-    <inertial>
-      <origin xyz="0 0 0" rpy="0 1.5707 1.5707"/>
-      <mass value="5"/>
-      <inertia
-        ixx=".1" ixy="0.0" ixz="0.0"
-        iyy=".1" iyz="0.0"
-        izz=".1"/>
+        <cylinder radius="0.125" length="0.150"/>
+      </geometry>
+    </visual>
+    <inertial>
+      <origin xyz="0 0 0" rpy="0 1.5707 1.5707"/>
+      <mass value="4"/>
+      <inertia
+        ixx="1" ixy="0.0" ixz="0.0"
+        iyy="1" iyz="0.0"
+        izz="1"/>
     </inertial>
   </link>
@@ -149,5 +149,5 @@
       <origin xyz="0 0 0" rpy="0 1.5707 1.5707"/>
       <geometry>
-        <cylinder radius="0.1" length="0.05"/>
+        <cylinder radius="0.125" length="0.150"/>
       </geometry>
     </collision>
@@ -155,18 +155,38 @@
       <origin xyz="0 0 0" rpy="0 1.5707 1.5707"/>
       <geometry>
-        <cylinder radius="0.1" length="0.05"/>
-      </geometry>
-    </visual>
-    <inertial>
-      <origin xyz="0 0 0" rpy="0 1.5707 1.5707"/>
-      <mass value="5"/>
-      <inertia
-        ixx=".1" ixy="0.0" ixz="0.0"
-        iyy=".1" iyz="0.0"
-        izz=".1"/>
-    </inertial>
+        <cylinder radius="0.125" length="0.150"/>
+      </geometry>
+    </visual>
+    <inertial>
+      <origin xyz="0 0 0" rpy="0 1.5707 1.5707"/>
+      <mass value="4"/>
+      <inertia
+        ixx="1" ixy="0.0" ixz="0.0"
+        iyy="1" iyz="0.0"
+        izz="1"/>
+    </inertial>
+  </link>
+  <link name="imu_link">
+   <inertial>
+    <mass value="0.001"/>
+    <origin rpy="0 0 0" xyz="0 0 0"/>
+    <inertia ixx="0.0001" ixy="0" ixz="0" iyy="0.000001" iyz="0" izz="0.0001"/>
+   </inertial>
+   <visual>
+    <origin rpy="0 0 0" xyz="0 0 0"/>
+    <geometry>
+      <box size="0.01 0.01 0.01"/>
+    </geometry>
+    <material name="red"/>
+   </visual>
+   <collision>
+    <origin rpy="0 0 0" xyz="0 0 0"/>
+    <geometry>
+      <box size=".01 .01 .01"/>
+    </geometry>
+   </collision>
   </link>
   <joint type="continuous" name="left_wheel_1_hinge">
-    <origin xyz="0.3 0.25 0" rpy="0 0 0"/>
+    <origin xyz="0.70 0.465 0.125" rpy="0 0 0"/>
     <!--origin xyz="0.1 0.13 0" rpy="0 1.5707 1.5707"/-->
     <child link="left_wheel_1"/>
@@ -177,5 +197,5 @@
   </joint>
   <joint type="continuous" name="left_wheel_2_hinge">
-    <origin xyz="0 0.25 0" rpy="0 0 0"/>
+    <origin xyz=" 0 0.465 0.125" rpy="0 0 0"/>
     <!--origin xyz="0.1 0.13 0" rpy="0 1.5707 1.5707"/-->
     <child link="left_wheel_2"/>
@@ -186,5 +206,5 @@
   </joint>
   <joint type="continuous" name="left_wheel_3_hinge">
-    <origin xyz="-0.3 0.25 0" rpy="0 0 0"/>
+    <origin xyz="-0.70 .48 0.125" rpy="0 0 0"/>
     <!--origin xyz="0.1 0.13 0" rpy="0 1.5707 1.5707"/-->
     <child link="left_wheel_3"/>
@@ -195,5 +215,5 @@
   </joint>
   <joint type="continuous" name="right_wheel_1_hinge">
-    <origin xyz="0.3 -0.25 0" rpy="0 0 0"/>
+    <origin xyz="0.70 -0.465 0.125" rpy="0 0 0"/>
     <!--origin xyz="0.1 -0.13 0" rpy="0 1.5707 1.5707"/-->
     <child link="right_wheel_1"/>
@@ -204,5 +224,5 @@
   </joint>
   <joint type="continuous" name="right_wheel_2_hinge">
-    <origin xyz="0 -0.25 0" rpy="0 0 0"/>
+    <origin xyz="0 -0.465 0.125" rpy="0 0 0"/>
     <!--origin xyz="0.1 -0.13 0" rpy="0 1.5707 1.5707"/-->
     <child link="right_wheel_2"/>
@@ -213,5 +233,5 @@
   </joint>
   <joint type="continuous" name="right_wheel_3_hinge">
-    <origin xyz="-0.3 -0.25 0" rpy="0 0 0"/>
+    <origin xyz="-0.70 -0.48 0.125" rpy="0 0 0"/>
     <!--origin xyz="0.1 -0.13 0" rpy="0 1.5707 1.5707"/-->
     <child link="right_wheel_3"/>
@@ -221,5 +241,11 @@
     <joint_properties damping="1.0" friction="1.0"/>
   </joint>
-  <link name="camera">
+  <joint name="imu_joint" type="fixed">
+    <axis xyz="0 0 1"/>
+    <origin xyz="0 0 0.3"/>
+    <parent link="chassis"/>
+    <child link="imu_link"/>
+  </joint>
+  <!--link name="camera">
     <collision>
       <origin xyz="0 0 0" rpy="0 0 0"/>
@@ -241,18 +267,18 @@
       <inertia ixx="1e-6" ixy="0" ixz="0" iyy="1e-6" iyz="0" izz="1e-6" />
     </inertial>
-  </link>
-  <joint name="camera_joint" type="fixed">
+  </link-->
+  <!--joint name="camera_joint" type="fixed">
     <axis xyz="0 1 0" />
     <origin xyz=".2 0 0" rpy="0 0 0"/>
     <parent link="chassis"/>
     <child link="camera"/>
-  </joint>
-  <joint name="hokuyo_joint" type="fixed">
+  </joint-->
+  <!--joint name="hokuyo_joint" type="fixed">
     <axis xyz="0 1 0" />
     <origin xyz=".15 0 0.15" rpy="0 0 0"/>
     <parent link="chassis"/>
     <child link="hokuyo"/>
-  </joint>
-  <!-- Hokuyo Laser -->
+  </joint-->
+  <!-- Hokuyo Laser >
   <link name="hokuyo">
     <collision>
@@ -273,32 +299,4 @@
       <inertia ixx="1e-6" ixy="0" ixz="0" iyy="1e-6" iyz="0" izz="1e-6" />
     </inertial>
-  </link>
- <link name='imu_link'>
-    <inertial>
-      <mass value="5"/>
-      <origin xyz="0.0 0 0.1" rpy=" 0 0 0"/>
-      <inertia
-          ixx="0.1" ixy="0" ixz="0"
-          iyy="0.1" iyz="0"
-          izz="0.1"
-      />
-    </inertial>
-    <collision name='collision'>
-      <geometry>
-        <cylinder radius="0.05" length="5.0"/>
-      </geometry>
-    </collision>
-    <visual name='imu_link_visual'>
-      <origin xyz="0 0 " rpy=" 0 0 0"/>
-      <geometry>
-        <cylinder radius="0.05" length="1.0"/>
-      </geometry>
-    </visual>
-  </link>
-<joint name="imu_link_joint" type="continuous">
-    <axis xyz="0 1 0" />
-    <origin xyz=".2 0 0" rpy="0 0 0"/>
-    <parent link="chassis"/>
-    <child link="imu_link"/>
-  </joint>
+  </link-->
 </robot>

Commit message: pushing latest code

File: src/mybot_ws/src/mybot_description/urdf/mybot.xacro (robot description, xacro)
@@ -187,4 +187,24 @@
    </collision>
   </link>
+  <link name="gps_link">
+   <inertial>
+    <mass value="0.001"/>
+    <origin rpy="0 0 0" xyz="0 0 0"/>
+    <inertia ixx="0.0001" ixy="0" ixz="0" iyy="0.000001" iyz="0" izz="0.0001"/>
+   </inertial>
+   <visual>
+    <origin rpy="0 0 0" xyz="0 0 0"/>
+    <geometry>
+      <box size="0.01 0.01 0.01"/>
+    </geometry>
+    <material name="red"/>
+   </visual>
+   <collision>
+    <origin rpy="0 0 0" xyz="0 0 0"/>
+    <geometry>
+      <box size=".01 .01 .01"/>
+    </geometry>
+   </collision>
+  </link>
   <joint type="continuous" name="left_wheel_1_hinge">
     <origin xyz="0.70 0.465 0.125" rpy="0 0 0"/>
@@ -246,4 +266,10 @@
     <parent link="chassis"/>
     <child link="imu_link"/>
+  </joint>
+  <joint name="gps_joint" type="fixed">
+    <axis xyz="0 0 1"/>
+    <origin xyz="0 0 0.3"/>
+    <parent link="chassis"/>
+    <child link="gps_link"/>
   </joint>
   <!--link name="camera">

Commit message: costmap issue solved

File: src/mybot_ws/src/mybot_description/urdf/mybot.xacro (robot description, xacro)
@@ -292,5 +292,5 @@
     </inertial>
   </link>
-  <joint name="laser_joint" type="fixed">
+  <joint name="laser_joint" type="continuous">
     <axis xyz="0 1 0" />
     <origin xyz=".15 0 0.15" rpy="0 0 0"/>
